File: hw/kicad/panel.kicad_sch (KiCad schematic)
At the start: 78 parts, among them J901 LCD ST7789, J911 ВХ1, J912 ВХ2, J913 ВЫХ, J914 ВЫХ2, SW900 EC11 МЕНЮ, SW901 EC11 ПАР.1, SW902 EC11 ПАР.2, SW903 EC11 ПАР.3, U901 MCP3208

Commit message: Reorganize KiCad schematic into 7 functional sheets with framed blocks
- Sheets: power, fpga, midi_sync, analog_in (inputs + ADC), audio_out
  (DAC + OUT/OUT2 + clip LEDs), phones, panel
- Each functional block is drawn in a dashed frame with a title; blocks are
  tiled across the sheet, A3/A2 chosen automatically
- Netlist check still 153/153; PDF and docs updated

Co-Authored-By: Claude Opus 5.5 <noreply@anthropic.com>
Claude-Session: https://claude.ai/code/session_01JcNV2ZCXWxtNzRVWffkrjk
Other:
- moved on the sheet: C901, C902, C903, C904, C905, C906, C907, C908, C909, C910, C911, C912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
