File: hw/kicad/power.kicad_sch (KiCad schematic)
At the start: 37 parts, among them J101 АВК-6 модуль, U101 LP5907MFX-3.3, U102 AP2112K-3.3, U103 AP2112K-3.3, U104 REF3025

Commit message: Reorganize KiCad schematic into 7 functional sheets with framed blocks
- Sheets: power, fpga, midi_sync, analog_in (inputs + ADC), audio_out
  (DAC + OUT/OUT2 + clip LEDs), phones, panel
- Each functional block is drawn in a dashed frame with a title; blocks are
  tiled across the sheet, A3/A2 chosen automatically
- Netlist check still 153/153; PDF and docs updated

Co-Authored-By: Claude Opus 5.5 <noreply@anthropic.com>
Claude-Session: https://claude.ai/code/session_01JcNV2ZCXWxtNzRVWffkrjk
Other:
- moved on the sheet: C101, C102, C103, C104, C105, C106, C107, C108, C109, C110, C111, C112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
